File: Ch1Power.kicad_sch (KiCad schematic)
At the start: 10 parts, among them J201 Banana_Red, J202 Banana_Black

Commit message: added loop calc
Other:
- sheet MCU ports: added Enable_DCDC, Enable_Linear; removed Enable
Changed lines of the file:
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@@
-	)
-	(junction
-		(at 76.2 104.14)
-		(diameter 0)
-		(color 0 0 0 0)
 	)
 	(junction
@@
 	(wire
 		(pts
-			(xy 180.34 120.65) (xy 76.2 120.65)
-		)
-		(stroke
-			(width 0)
-			(type default)
-		)
-	)
-	(wire
-		(pts
 			(xy 199.39 80.01) (xy 105.41 80.01)
 		)
@@
 	(wire
 		(pts
+			(xy 66.04 120.65) (xy 180.34 120.65)
+		)
+		(stroke
+			(width 0)
+			(type default)
+		)
+	)
+	(wire
+		(pts
 			(xy 110.49 90.17) (xy 110.49 82.55)
 		)
@@
 	(wire
 		(pts
-			(xy 76.2 104.14) (xy 90.17 104.14)
+			(xy 66.04 104.14) (xy 90.17 104.14)
 		)
 		(stroke
@@
 	(wire
 		(pts
-			(xy 66.04 104.14) (xy 76.2 104.14)
-		)
-		(stroke
-			(width 0)
-			(type default)
-		)
-	)
-	(wire
-		(pts
 			(xy 25.4 77.47) (xy 90.17 77.47)
 		)
@@
 		(pts
 			(xy 156.21 107.95) (xy 180.34 107.95)
-		)
-		(stroke
-			(width 0)
-			(type default)
-		)
-	)
-	(wire
-		(pts
-			(xy 76.2 120.65) (xy 76.2 104.14)
 		)
 		(stroke
@@
 			)
 		)
-		(pin "Enable" output
-			(at 66.04 104.14 0)
-			(effects
-				(font
-					(size 1.27 1.27)
-				)
-				(justify right)
-			)
-		)
 		(pin "SPI_ADC_CS" output
 			(at 66.04 133.35 0)
@@
 			(effects
 				(font
+					(size 1.27 1.27)
+				)
+				(justify right)
+			)
+		)
+		(pin "Enable_DCDC" output
+			(at 66.04 104.14 0)
+			(effects
+				(font
+					(size 1.27 1.27)
+				)
+				(justify right)
+			)
+		)
+		(pin "Enable_Linear" output
+			(at 66.04 120.65 0)
+			(effects
+				(font
