File: MCU.kicad_sch (KiCad schematic)
At the start: 19 parts, among them J801 Conn_01x03_Pin, J802 Conn_02x02_Odd_Even, Q801 BSS138, Q802 BSS138, U801 ISO6721RFBD, U802 ATtiny1614-SS

Commit message: changed pass element drive
Parts:
- added C805: 100n, Capacitor_SMD:C_0603_1608Metric, symbol Device:C
Connections:
- net +3.3V: now reaches U801.1 (VCC1)
- net +3.3V: now also C805.1
- net Tx_Ctr: now reaches U801.2 (INA)
- net Rx_Ctr: now reaches U801.3 (OUTB)
- net GNDD: now reaches U801.4 (GND1)
- net GNDD: now also C805.2
