File: DAC_ADC.kicad_sch (KiCad schematic)
At the start: 8 parts, among them U701 ADS1118IDGS, U702 MCP48FVB22

Commit message: added Ch2 and removed global power flags
Connections:
- net CH1_+3.3V renamed +3V3
- net GND1 renamed GND
