File: MCU2.kicad_sch (KiCad schematic)
At the start: 20 parts, among them J801 Conn_01x03_Pin, J802 Conn_02x02_Odd_Even, Q801 BSS138, Q802 BSS138, U801 ISO6721RFBD, U802 ATtiny1614-SS

Commit message: added Ch2 and removed global power flags
Parts:
- removed C801, C802, C803, C805: 100n, Capacitor_SMD:C_0603_1608Metric, symbol Device:C
- removed C804: 1u, Capacitor_SMD:C_0603_1608Metric, symbol Device:C
- removed D801, D802: LED 3V3, LED_SMD:LED_0603_1608Metric, symbol Device:LED
- removed J801: Conn_01x03_Pin, Connector_JST:JST_SH_BM03B-SRSS-TB_1x03-1MP_P1.00mm_Vertical, symbol Connector:Conn_01x03_Pin
- removed J802: Conn_02x02_Odd_Even, Connector_PinHeader_2.00mm:PinHeader_2x02_P2.00mm_Horizontal, symbol Connector_Generic:Conn_02x02_Odd_Even
- removed Q801, Q802: BSS138, Package_TO_SOT_SMD:SOT-23, symbol Transistor_FET:BSS138
- removed R801, R802: 10k, Resistor_SMD:R_0603_1608Metric, symbol Device:R
- removed R803, R806: 2,4k, Resistor_SMD:R_0603_1608Metric, symbol Device:R
- removed R804, R805: 1k, Resistor_SMD:R_0603_1608Metric, symbol Device:R
- removed TH801: NCU18XH103F60RB, Resistor_SMD:R_0603_1608Metric, symbol Device:Thermistor_NTC
- removed U801: ISO6721RFBD, Package_SO:SOIC-8_3.9x4.9mm_P1.27mm, symbol Isolator:ISO6721RFBD
- removed U802: ATtiny1614-SS, Package_SO:SOIC-14_3.9x8.7mm_P1.27mm, symbol MCU_Microchip_ATtiny:ATtiny1614-SS
- added C1201, C1202, C1203, C1205: 100n, Capacitor_SMD:C_0603_1608Metric, symbol Device:C
- added C1204: 1u, Capacitor_SMD:C_0603_1608Metric, symbol Device:C
- added D1201, D1202: LED 3V3, LED_SMD:LED_0603_1608Metric, symbol Device:LED
- added J1201: Conn_01x03_Pin, Connector_JST:JST_SH_BM03B-SRSS-TB_1x03-1MP_P1.00mm_Vertical, symbol Connector:Conn_01x03_Pin
- added J1202: Conn_02x02_Odd_Even, Connector_PinHeader_2.00mm:PinHeader_2x02_P2.00mm_Horizontal, symbol Connector_Generic:Conn_02x02_Odd_Even
- added Q1201, Q1202: BSS138, Package_TO_SOT_SMD:SOT-23, symbol Transistor_FET:BSS138
- added R1201, R1202: 10k, Resistor_SMD:R_0603_1608Metric, symbol Device:R
- added R1203, R1206: 2,4k, Resistor_SMD:R_0603_1608Metric, symbol Device:R
- added R1204, R1205: 1k, Resistor_SMD:R_0603_1608Metric, symbol Device:R
- added TH1201: NCU18XH103F60RB, Resistor_SMD:R_0603_1608Metric, symbol Device:Thermistor_NTC
- added U1201: ISO6721RFBD, Package_SO:SOIC-8_3.9x4.9mm_P1.27mm, symbol Isolator:ISO6721RFBD
- added U1202: ATtiny1614-SS, Package_SO:SOIC-14_3.9x8.7mm_P1.27mm, symbol MCU_Microchip_ATtiny:ATtiny1614-SS
Connections:
- net +3.3V: now also C1201.1, U1201.1 (VCC1)
- net CC/~{CV}: now also R1205.1
- net DAC_LAT: now also U1202.4 (PA6)
- net Enable: now also R1203.1, R1204.1, U1202.3 (PA5)
- net GNDD: now also C1201.2, U1201.4 (GND1)
- net NTC1: now also C1204.1, R1202.2, U1202.9 (PB0)
- net Rx: now also U1201.7 (OUTA), U1202.6 (PB3)
- net Rx_Ctr: now also U1201.3 (OUTB)
- net SPI_ADC_CS: now also U1202.2 (PA4)
- net SPI_DAC_CS: now also U1202.5 (PA7)
- net SPI_MISO: now also U1202.12 (PA2)
- net SPI_MOSI: now also U1202.11 (PA1)
- net SPI_SCK: now also U1202.13 (PA3)
- net Tx: now also U1201.6 (INB), U1202.7 (PB2)
- net Tx_Ctr: now also U1201.2 (INA)
- net UPDI: now also J1201.1 (Pin_1), U1202.10 (~{RESET}/PA0)
- net ~{LED_CC}: now also D1202.1 (K), J1202.3 (Pin_3), Q1202.3 (D)
- net ~{LED_Enable}: now also J1202.1 (Pin_1), Q1201.3 (D)
- new net: R1201.2, R1202.1, TH1201.1
- new net: Q1201.1 (G), R1204.2
- new net: Q1202.1 (G), R1205.2
- new net: D1201.2 (A), R1203.2
- new net: D1202.2 (A), R1206.2
- new net CH2_+3.3V: C1202.1, C1203.1, C1205.1, J1201.2 (Pin_2), J1202.4 (Pin_4), R1201.1, R1206.1, U1201.8 (VCC2), U1202.1 (VCC)
- new net GND2: C1202.2, C1203.2, C1204.2, C1205.2, D1201.1 (K), J1201.3 (Pin_3), Q1201.2 (S), Q1202.2 (S), TH1201.2, U1201.5 (GND2), U1202.14 (GND)
