File: Power.kicad_sch (KiCad schematic)
At the start: 22 parts, among them U1001 AP64060QWU, U1002 AP7383, U1003 LM2776, U1004 XC6901D121MR-G

Commit message: routing
Parts:
- removed C1004: 56p, Capacitor_SMD:C_0603_1608Metric, symbol Device:C
- removed U1001: AP64060QWU, Package_TO_SOT_SMD:TSOT-23-6, symbol Regulator_Switching:AP63200WU
- added U601: LMR51606, Package_TO_SOT_SMD:SOT-23-6, symbol eiene Symbole:LMR51606
- L1001: value 10u CBC3225T100KR -> 33u VLS6045EX-330M; footprint Inductor_SMD:L_1210_3225Metric -> Inductor_SMD:L_TDK_VLS6045EX_VLS6045AF
- R1001: value 115k -> 75k
- R1002: value 22,1k -> 16,2k
Connections:
- net 40V: now also U601.4 (EN), U601.5 (VIN)
- net GND: now also U601.2 (GND)
- net SW: now also U601.6 (SW)
- net at R1001.2, R1002.1: now also U601.3 (FB)
- net at C1003.1: now also U601.1 (CB)
Other:
- note added: "4,5V"
- note removed: "5V"
- moved on the sheet: C1003

Commit message: added loop calc
Parts:
- added TP603, TP604: TestPoint_Alt, TestPoint:TestPoint_Keystone_5005-5009_Compact, symbol Connector:TestPoint_Alt
- added TP605, TP606, TP607: TestPoint, LibEigen:SMD Test Point PCWCTE, symbol Connector:TestPoint
- added TP608: TestPoint_Alt, TestPoint:TestPoint_Pad_D1.0mm, symbol Connector:TestPoint_Alt
Connections:
- net +3V3: now also TP606.1
- net -1V2: now also TP607.1
- net 5V: now also TP605.1
- net GND: now also TP603.1, TP604.1
- net at C1010.1, D1002.1 (K), U1003.1 (VOUT)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: now also TP608.1

Commit message: add diodes for clamping
Parts:
- added TP602: TestPoint_Alt, TestPoint:TestPoint_Keystone_5005-5009_Compact, symbol Connector:TestPoint_Alt
Connections:
- net +3V3: now also TP602.1
Changed lines of the file:
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@@
+	)
+	(junction
+		(at 195.58 24.13)
+		(diameter 0)
+		(color 0 0 0 0)
 	)
 	(junction
@@
 	(wire
 		(pts
-			(xy 198.12 24.13) (xy 185.42 24.13)
+			(xy 198.12 24.13) (xy 195.58 24.13)
 		)
 		(stroke
@@
 		(pts
 			(xy 96.52 26.67) (xy 106.68 26.67)
+		)
+		(stroke
+			(width 0)
+			(type default)
+		)
+	)
+	(wire
+		(pts
+			(xy 195.58 24.13) (xy 185.42 24.13)
 		)
 		(stroke
@@
 					(unit 1)
 				)
+			)
+		)
+	)
+	(symbol
+		(lib_id "Connector:TestPoint_Alt")
+		(at 195.58 24.13 0)
+		(unit 1)
+		(body_style 1)
+		(exclude_from_sim no)
+		(in_bom yes)
+		(on_board yes)
+		(in_pos_files yes)
+		(dnp no)
+		(fields_autoplaced yes)
+		(property "Reference" "TP602"
+			(at 198.12 19.5579 0)
+			(show_name no)
+			(do_not_autoplace no)
+			(effects
+				(font
+					(size 1.27 1.27)
+				)
+				(justify left)
+			)
+		)
+		(property "Value" "TestPoint_Alt"
+			(at 198.12 22.0979 0)
+			(show_name no)
+			(do_not_autoplace no)
+			(effects
+				(font
+					(size 1.27 1.27)
+				)
+				(justify left)
+			)
+		)
+		(property "Footprint" "TestPoint:TestPoint_Keystone_5005-5009_Compact"
+			(at 200.66 24.13 0)
+			(hide yes)
+			(show_name no)
+			(do_not_autoplace no)
+			(effects
+				(font
+					(size 1.27 1.27)
+				)
+			)
+		)
+		(property "Datasheet" ""
+			(at 200.66 24.13 0)
+			(hide yes)
+			(show_name no)
+			(do_not_autoplace no)
+			(effects
+				(font
+					(size 1.27 1.27)
+				)
+			)
+		)
+		(property "Description" "test point (alternative shape)"
+			(at 195.58 24.13 0)
+			(hide yes)
+			(show_name no)
+			(do_not_autoplace no)
+			(effects
+				(font
+					(size 1.27 1.27)
+				)
+			)
+		)
+		(pin "1"
+		)
+		(instances
+			(project "DualPreRegPowerSupply"
+				(path "/6e74608c-23b9-4b98-8fc4-fa8fd655ae50/19bfe284-0b9b-4876-b680-4ee0d6ee0ed7/1e97c929-9584-4135-ba9a-4ad49b795d46"
+					(reference "TP602")
+					(unit 1)
+				)
+				(path "/6e74608c-23b9-4b98-8fc4-fa8fd655ae50/343e6ab8-61bf-4409-bd59-a9fdebf952af/1e97c929-9584-4135-ba9a-4ad49b795d46"
+					(reference "TP1507")
+					(unit 1)
+				)
