File: hardware/Digi_Power.kicad_sch (KiCad schematic)
At the start: 18 parts, among them J901 Power Input, U901 AP63200WU

Commit message: routing
Parts:
- D901: value SM6T36A -> SMBJ12A
Changed lines of the file:
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@@
 			)
 		)
-		(property "Value" "SM6T36A"
+		(property "Value" "SMBJ12A"
 			(at 59.69 34.2899 90)
 			(show_name no)
