File: hardware/Ch1Power.kicad_sch (KiCad schematic)
At the start: 10 parts, among them J201 Banana_Red, J202 Banana_Black

Commit message: routing
Parts:
- D201: value SM6T36A -> SMBJ36A
Changed lines of the file:
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@@
 			)
 		)
-		(property "Value" "SM6T36A"
+		(property "Value" "SMBJ36A"
 			(at 254 113.0299 90)
 			(show_name no)
