File: hardware/Control.kicad_sch (KiCad schematic)
At the start: 15 parts, among them J204 Conn_02x05_Odd_Even, J401 Conn_02x05_Odd_Even, M401 Fan_4pin, U401 TMP1075D

Commit message: routing
Parts:
- removed J401: Conn_02x05_Odd_Even, Connector_PinHeader_2.00mm:PinHeader_2x05_P2.00mm_Horizontal, symbol Connector_Generic:Conn_02x05_Odd_Even
- added J203: Conn_02x04_Odd_Even, Connector_PinHeader_2.54mm:PinHeader_2x04_P2.54mm_Horizontal, symbol Connector_Generic:Conn_02x04_Odd_Even
- added J205: Conn_01x04_Pin, Connector_PinHeader_2.54mm:PinHeader_1x04_P2.54mm_Vertical, symbol Connector:Conn_01x04_Pin
Connections:
- net +3.3V: now also J203.3 (Pin_3)
- net CS: now also J203.1 (Pin_1)
- net DC: now also J205.1 (Pin_1)
- net GNDD: now also J203.5 (Pin_5)
- net RESET: now also J205.4 (Pin_4)
- net SCK: now also J205.3 (Pin_3)
- net SCL: now also J203.8 (Pin_8)
- net SDA: now also J203.6 (Pin_6)
- net SDI(MOSI): now also J205.2 (Pin_2)
- net ~{INT}: now also J203.7 (Pin_7)
- net ROT_A: now reaches A401.14 (GPIO14)
- net ROT_A: now also J203.2 (Pin_2)
- net ROT_B: now reaches A401.15 (GPIO15)
- net ROT_B: now also J203.4 (Pin_4)
Other:
- note added: "1001111"
