File: hardware/DualPreRegPowerSupply.kicad_pcb (KiCad board)
At the start: 4 copper layers, 100 x 100 mm, 349 parts, among them J101 Power Input, J102 Conn_01x03_Pin, J103 Conn_02x02_Odd_Even, J201 Banana_Red, J202 Banana_Black, J204 Conn_02x05_Odd_Even, J401 Conn_02x05_Odd_Even, J402 Banana_Red, J403 Banana_Black, J601 Power Input, J801 Conn_01x03_Pin, J802 Conn_02x02_Odd_Even, J901 Power Input, M401 Fan_4pin, Q101 MMBT3906, Q102 BCP56, Q103 BSS138, Q104 TIP125, Q105 BSS138, Q106 BSS138, Q107 BCP56, Q301 BCP56, Q302 BSS138, Q303 TIP125, Q304 BCP56, Q501 MMBT3906, Q801 BSS138, Q802 BSS138, U1002 AP7383, U1003 LM2776, U1004 XC6901D121MR-G, U101 TLV4387PWR, U102 ISO6721RFBD, U104 LT8612, U105 LMV331, U106 ATtiny1614-SS, U107 ADS1118IDGS, U108 MCP48FVB22, U109 AP7383, U110 LM2776, U111 XC6901D121MR-G, U1501 LMR51606, U301 TLV4387PWR, U302 LMV331, U401 TMP1075D, U501 LT8612, U601 LMR51606, U701 ADS1118IDGS, U702 MCP48FVB22, U801 ISO6721RFBD, U802 ATtiny1614-SS, U901 AP63200WU

Commit message: routing
Parts:
- removed D102, D301: BAT54A, Package_TO_SOT_SMD:SOT-23-3
- added D1006: 1N4148WS, Diode_SMD:D_SOD-323, B.Cu at (127.7, 120.3)
- added D1007: 1N4148WS, Diode_SMD:D_SOD-323, B.Cu at (117.8, 113.0)
- added D1008: 1N4148WS, Diode_SMD:D_SOD-323, B.Cu at (117.8, 115.0)
- added D1204: 1N4148WS, Diode_SMD:D_SOD-323, B.Cu at (171.5, 121.6)
- added D1205: 1N4148WS, Diode_SMD:D_SOD-323, B.Cu at (179.8, 120.0)
- added D1206: 1N4148WS, Diode_SMD:D_SOD-323, B.Cu at (181.8, 120.0)
- D1201, D1202, D1203: moved to B.Cu
- D901: value SM6T36A -> SMBJ12A
- Q102, Q107, TP402, TP403: moved to F.Cu
- R130, R508: value 100k -> 62k
- moved C145 131.9 mm to (161.6, 140.3), turned to 180 degrees
- moved R141 130.0 mm to (161.6, 142.7), turned to 180 degrees
- moved Q107 124.0 mm to (167.4, 121.2)
- moved TP403 116.0 mm to (152.0, 133.6), turned to 0 degrees
- moved Q102 109.7 mm to (174.9, 121.2)
- moved TP104 109.6 mm to (177.9, 120.1), turned to 0 degrees
- moved F102 107.8 mm to (172.2, 127.1)
- moved C107 107.1 mm to (184.2, 59.9), turned to 180 degrees
- moved L101 106.4 mm to (189.3, 64.4), turned to 0 degrees
- moved C105 106.4 mm to (184.2, 57.5), turned to 180 degrees
- moved R115 104.6 mm to (180.9, 62.3)
- moved R114 104.4 mm to (180.9, 59.2)
- moved TP105 103.8 mm to (182.3, 106.2), turned to 0 degrees
- moved R123 103.4 mm to (175.5, 124.3), turned to 180 degrees
- moved R129 103.3 mm to (176.5, 118.0), turned to 0 degrees
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Connections:
- J103 pad 2: unconnected-(J103-Pin_2-Pad2) -> +3V3Ch2
- J802 pad 2: unconnected-(J802-Pin_2-Pad2) -> +3V3Ch1
- Q107 pad 2: /Ch1Power1/Linear_PostReg/preFuseOut+ -> Net-(D1204-K)
- Q107 pad 4: /Ch1Power1/Linear_PostReg/preFuseOut+ -> Net-(D1204-K)
- Q304 pad 2: /Ch1Power/Linear_PostReg/preFuseOut+ -> Net-(D1006-K)
- Q304 pad 4: /Ch1Power/Linear_PostReg/preFuseOut+ -> Net-(D1006-K)
Routing:
- net /Ch1Power1/Linear_PostReg/OUT+: track 0.00 -> 147.0 mm, vias 0 -> 3
- net /Ch1Power1/Linear_PostReg/OUT-: track 0.00 -> 129.3 mm, vias 0 -> 1
- net -1V2Ch2: track 0.00 -> 111.7 mm, vias 0 -> 4
- net /Ch1Power1/Linear_PostReg/OE: track 0.00 -> 71.9 mm, vias 0 -> 2
- net /Ch1Power1/Linear_PostReg/PreReg: track 0.00 -> 48.8 mm, vias 0 -> 4
- net GND_Ch2: track 4.83 -> 46.8 mm, vias 36 -> 127
- net +40VCh2: track 0.00 -> 41.6 mm
- net /Ch1Power1/Power/5V: track 0.00 -> 36.0 mm, vias 0 -> 4
- net /Ch1Power1/Rx_Ctr: track 0.00 -> 32.8 mm, vias 0 -> 2
- net /Ch1Power1/Linear_PostReg/CC/~{CV}: track 0.00 -> 30.2 mm
- net /Ch1Power1/Tx_Ctr: track 0.00 -> 29.0 mm, vias 0 -> 2
- net /Ch1Power1/DCDCTracking/DCDC_FB: track 0.71 -> 28.8 mm, vias 1 -> 2
- net +3V3Ch2: track 2.09 -> 27.2 mm, vias 1 -> 22
- net /Ch1Power1/MCU/NTC1: track 0.00 -> 23.3 mm
- net /Ch1Power1/DCDCTracking/Enable: track 3.03 -> 25.5 mm, vias 1 -> 2
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- added copper zone on B.Cu, net +3V3Ch2
- added copper zone on B.Cu, net /Ch1Power1/Linear_PostReg/OUT-
- added copper zone on B.Cu, net /Ch1Power1/Linear_PostReg/PreReg
- added copper zone on B.Cu, net /Ch1Power1/Power/5V
- added copper zone on B.Cu, net /Ch1Power1/Power/SW
- removed copper zone on F.Cu, net /Ch1Power/Linear_PostReg/preFuseOut+

Commit message: routing
Parts:
- removed J401: Conn_02x05_Odd_Even, Connector_PinHeader_2.00mm:PinHeader_2x05_P2.00mm_Horizontal
- added J203: Conn_02x04_Odd_Even, Connector_PinHeader_2.54mm:PinHeader_2x04_P2.54mm_Horizontal, F.Cu at (143.3, 132.0)
- added J205: Conn_01x04_Pin, Connector_PinHeader_2.54mm:PinHeader_1x04_P2.54mm_Vertical, F.Cu at (143.3, 129.5)
- J103, J802: footprint Connector_PinHeader_2.00mm:PinHeader_2x02_P2.00mm_Horizontal -> Connector_PinHeader_2.54mm:PinHeader_2x02_P2.54mm_Horizontal
- moved R140 10.5 mm to (164.1, 123.1), turned to 180 degrees
- moved Q801 10.4 mm to (112.7, 124.6)
- moved R804 8.07 mm to (117.2, 124.7)
- moved D107 6.45 mm to (163.3, 125.5), turned to 90 degrees
- moved J103 3.96 mm to (162.8, 132.0)
- moved J802 3.96 mm to (118.8, 132.0)
- moved C202 3.95 mm to (139.4, 137.2)
- moved C145 3.20 mm to (161.5, 137.1)
- moved R141 3.20 mm to (161.5, 139.5)
- moved C309 2.80 mm to (117.5, 140.1)
- moved R319 2.70 mm to (117.5, 137.7)
Connections:
- A401 pad 14: unconnected-(A401-GPIO14-Pad14) -> /Control/ROT_A
- A401 pad 15: unconnected-(A401-GPIO15-Pad15) -> /Control/ROT_B
Routing:
- net /Control/ROT_B: track 0.00 -> 32.7 mm, vias 0 -> 1
- net /Control/ROT_A: track 0.00 -> 29.7 mm, vias 0 -> 1
- net /Ch1Power/Linear_PostReg/OE: track 64.2 -> 54.7 mm
- net /Control/DC: track 26.6 -> 17.4 mm
- net /Control/SDI(MOSI): track 25.7 -> 16.7 mm
- net /Control/SCK: track 25.1 -> 16.3 mm
- net /Control/RESET: track 23.8 -> 15.2 mm
- net /Ch1Power/MCU/~{LED_Enable}: track 2.73 -> 10.9 mm
- net /Control/CS: track 28.6 -> 22.8 mm
- net Net-(Q801-G): track 2.32 -> 6.30 mm
- net /Ch1Power/Linear_PostReg/OUT+: track 92.8 -> 89.4 mm
- net /Ch1Power1/MCU/~{LED_Enable}: track 7.50 -> 4.18 mm
- net /Control/~{INT}: track 20.6 -> 17.4 mm
- net +3.3V: track 30.2 -> 27.4 mm
- net GNDD: track 32.5 -> 29.6 mm
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