File: hardware/Input.kicad_sch (KiCad schematic)
At the start: 11 parts, among them J601 Power Input

Commit message: routing
Parts:
- D601: value SM6T36A -> SMBJ40A
Changed lines of the file:
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@@
 			)
 		)
-		(property "Value" "SM6T36A"
+		(property "Value" "SMBJ40A"
 			(at 116.84 106.6799 90)
 			(show_name no)
