File: hardware/MCU.kicad_sch (KiCad schematic)
At the start: 20 parts, among them J801 Conn_01x03_Pin, J802 Conn_02x02_Odd_Even, Q801 BSS138, Q802 BSS138, U801 ISO6721RFBD, U802 ATtiny1614-SS

Commit message: routing
Connections:
- net +3V3: now also J802.2 (Pin_2)
Changed lines of the file:
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@@
+	(wire
+		(pts
+			(xy 250.19 105.41) (xy 242.57 105.41)
+		)
+		(stroke
+			(width 0)
+			(type default)
+		)
+	)
 	(wire
 		(pts
@@
 		)
 	)
+	(label "+3V3"
+		(at 250.19 105.41 180)
+		(effects
+			(font
+				(size 1.27 1.27)
+			)
+			(justify right bottom)
+		)
+	)

Commit message: routing
Parts:
- J802: footprint Connector_PinHeader_2.00mm:PinHeader_2x02_P2.00mm_Horizontal -> Connector_PinHeader_2.54mm:PinHeader_2x02_P2.54mm_Horizontal
Changed lines of the file:
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@@
 			)
 		)
-		(property "Footprint" "Connector_PinHeader_2.00mm:PinHeader_2x02_P2.00mm_Horizontal"
+		(property "Footprint" "Connector_PinHeader_2.54mm:PinHeader_2x02_P2.54mm_Horizontal"
 			(at 234.95 105.41 0)
 			(hide yes)
