File: hardware_main/DAC_ADC.kicad_sch (KiCad schematic)
At the start: 8 parts, among them U701 ADS1118IDGS, U702 MCP48FVB22

Commit message: routing
Parts:
- C701, C702: value ## -> 4,7u
- R701, R702: value ## -> 1k
Other:
- note added: "0V - 2,44V"
- note added: "33 Hz LPF"
- note added: "Iout = Iset * 1/12"
- note added: "Vout = Vset * 15"
Changed lines of the file:
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@@
 	(generator_version "10.0")
 	(paper "A4")
+	(text "0V - 2,44V"
+		(exclude_from_sim no)
+		(at 167.64 114.3 0)
+		(effects
+			(font
+				(size 1.27 1.27)
+			)
+		)
+	)
+	(text "33 Hz LPF"
+		(exclude_from_sim no)
+		(at 92.71 34.29 0)
+		(effects
+			(font
+				(size 1.27 1.27)
+			)
+		)
+	)
+	(text "Iout = Iset * 1/12"
+		(exclude_from_sim no)
+		(at 162.56 120.65 0)
+		(effects
+			(font
+				(size 1.27 1.27)
+			)
+			(justify left top)
+		)
+	)
+	(text "Vout = Vset * 15"
+		(exclude_from_sim no)
+		(at 162.56 106.68 0)
+		(effects
+			(font
+				(size 1.27 1.27)
+			)
+			(justify left top)
+		)
+	)
+	(text "33 Hz LPF"
+		(exclude_from_sim no)
+		(at 93.98 52.07 0)
+		(effects
+			(font
+				(size 1.27 1.27)
+			)
+		)
+	)
 	(junction
 		(at 91.44 36.83)
@@
 			)
 		)
-		(property "Value" "##"
+		(property "Value" "1k"
 			(at 83.82 50.8 90)
 			(show_name no)
@@
 			)
 		)
-		(property "Value" "##"
+		(property "Value" "1k"
 			(at 83.82 33.02 90)
 			(show_name no)
@@
 			)
 		)
-		(property "Value" "##"
+		(property "Value" "4,7u"
 			(at 95.25 60.9599 0)
 			(show_name no)
@@
 			)
 		)
-		(property "Value" "##"
+		(property "Value" "4,7u"
 			(at 95.25 43.1799 0)
 			(show_name no)
