File: hardware_main/DAC_ADC.kicad_sch (KiCad schematic)
At the start: 8 parts, among them U701 ADS1118IDGS, U702 MCP48FVB22

Commit message: stability calc
Parts:
- added C806, C807: 4,7u, Capacitor_SMD:C_0603_1608Metric, symbol Device:C
- added R807, R808: 1k, Resistor_SMD:R_0603_1608Metric, symbol Device:R
Connections:
- net GND: now also C806.2, C807.2
- net Iset: now also C807.1, R808.1; no longer U702.5 (VB)
- net Vset: now also C806.1, R807.1; no longer U702.4 (VA)
- new net: R808.2, U702.5 (VB)
- new net: R807.2, U702.4 (VA)

Commit message: calc and cleanup
Parts:
- added C808: 10u, Capacitor_SMD:C_0805_2012Metric, symbol Device:C
- C806: value 4,7u -> 100n
- C807: value 4,7u -> 27n
- R807: value 1k -> 12k
- R808: value 1k -> 10k
Connections:
- net +3V3: now also C808.1
- net GND: now also C808.2
Other:
- note added: "Iout = Iset * 1/1,2 2,44 / 1,2 = 2,0333A"
- note added: "Vout = Vset * 15 2,44 * 15 = 36,6V"
- note added: "τ = 9 us"
- note removed: "Iout = Iset * 1/12"
- note removed: "Vout = Vset * 15"
- moved on the sheet: C704
Changed lines of the file:
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@@
+		)
+	)
+	(text "τ = 9 us"
+		(exclude_from_sim no)
+		(at 205.74 123.19 0)
+		(effects
+			(font
+				(size 1.27 1.27)
+			)
 		)
 	)
@@
 		)
 	)
-	(text "Iout = Iset * 1/12"
+	(text "Iout = Iset * 1/1,2\n2,44 / 1,2 = 2,0333A"
 		(exclude_from_sim no)
-		(at 160.02 130.81 0)
+		(at 161.29 127 0)
 		(effects
 			(font
@@
 		)
 	)
-	(text "Vout = Vset * 15"
+	(text "Vout = Vset * 15\n2,44 * 15 = 36,6V"
 		(exclude_from_sim no)
 		(at 162.56 102.87 0)
@@
 	(wire
 		(pts
-			(xy 151.13 170.18) (xy 151.13 165.1)
+			(xy 149.86 158.75) (xy 149.86 153.67)
 		)
 		(stroke
@@
 	(wire
 		(pts
-			(xy 151.13 152.4) (xy 151.13 157.48)
+			(xy 149.86 140.97) (xy 149.86 146.05)
 		)
 		(stroke
@@
 	(wire
 		(pts
+			(xy 124.46 140.97) (xy 124.46 146.05)
+		)
+		(stroke
+			(width 0)
+			(type default)
+		)
+	)
+	(wire
+		(pts
 			(xy 182.88 110.49) (xy 182.88 104.14)
 		)
@@
 	(wire
 		(pts
+			(xy 124.46 158.75) (xy 124.46 153.67)
+		)
+		(stroke
+			(width 0)
+			(type default)
+		)
+	)
+	(wire
+		(pts
 			(xy 149.86 133.35) (xy 149.86 128.27)
 		)
@@
 	)
 	(label "+3V3"
-		(at 151.13 152.4 270)
+		(at 149.86 140.97 270)
 		(effects
 			(font
@@
 		)
 	)
+	(label "+3V3"
+		(at 124.46 140.97 270)
+		(effects
+			(font
+				(size 1.27 1.27)
+			)
+			(justify right bottom)
+		)
+	)
 	(label "GND"
 		(at 200.66 118.11 90)
@@
 	)
 	(label "GND"
-		(at 151.13 170.18 90)
+		(at 124.46 158.75 90)
+		(effects
+			(font
+				(size 1.27 1.27)
+			)
+			(justify left bottom)
+		)
+	)
+	(label "GND"
+		(at 149.86 158.75 90)
 		(effects
 			(font
@@
 	(symbol
 		(lib_id "Device:C")
-		(at 151.13 161.29 0)
+		(at 149.86 149.86 0)
 		(unit 1)
 		(body_style 1)
@@
 		(fields_autoplaced yes)
 		(property "Reference" "C704"
-			(at 154.94 160.0199 0)
+			(at 153.67 148.5899 0)
 			(show_name no)
 			(do_not_autoplace no)
@@
 		)
 		(property "Value" "100n"
-			(at 154.94 162.5599 0)
+			(at 153.67 151.1299 0)
 			(show_name no)
 			(do_not_autoplace no)
@@
 		)
 		(property "Footprint" "Capacitor_SMD:C_0603_1608Metric"
-			(at 152.0952 165.1 0)
+			(at 150.8252 153.67 0)
 			(hide yes)
 			(show_name no)
@@
 		)
 		(property "Datasheet" ""
-			(at 151.13 161.29 0)
+			(at 149.86 149.86 0)
 			(hide yes)
 			(show_name no)
@@
 		)
 		(property "Description" "Unpolarized capacitor"
-			(at 151.13 161.29 0)
+			(at 149.86 149.86 0)
 			(hide yes)
 			(show_name no)
@@
 			)
 		)
-		(property "Value" "1k"
+		(property "Value" "10k"
 			(at 193.04 120.65 90)
 			(show_name no)
@@
 			)
 		)
-		(property "Value" "1k"
+		(property "Value" "12k"
 			(at 193.04 100.33 90)
 			(show_name no)
@@
 	(symbol
 		(lib_id "Device:C")
+		(at 124.46 149.86 0)
+		(unit 1)
+		(body_style 1)
+		(exclude_from_sim no)
+		(in_bom yes)
+		(on_board yes)
+		(in_pos_files yes)
+		(dnp no)
+		(fields_autoplaced yes)
+		(property "Reference" "C808"
+			(at 128.27 148.5899 0)
+			(show_name no)
+			(do_not_autoplace no)
+			(effects
+				(font
+					(size 1.27 1.27)
+				)
+				(justify left)
+			)
+		)
+		(property "Value" "10u"
+			(at 128.27 151.1299 0)
+			(show_name no)
+			(do_not_autoplace no)
+			(effects
+				(font
+					(size 1.27 1.27)
+				)
+				(justify left)
+			)
+		)
+		(property "Footprint" "Capacitor_SMD:C_0805_2012Metric"
+			(at 125.4252 153.67 0)
+			(hide yes)
+			(show_name no)
+			(do_not_autoplace no)
+			(effects
+				(font
+					(size 1.27 1.27)
+				)
+			)
+		)
+		(property "Datasheet" ""
+			(at 124.46 149.86 0)
+			(hide yes)
+			(show_name no)
+			(do_not_autoplace no)
+			(effects
+				(font
+					(size 1.27 1.27)
+				)
+			)
+		)
+		(property "Description" "Unpolarized capacitor"
+			(at 124.46 149.86 0)
+			(hide yes)
+			(show_name no)
+			(do_not_autoplace no)
+			(effects
+				(font
+					(size 1.27 1.27)
+				)
+			)
+		)
+		(pin "1"
+		)
+		(pin "2"
+		)
+		(instances
+			(project "DualPreRegPowerSupply"
+				(path "/6e74608c-23b9-4b98-8fc4-fa8fd655ae50/19bfe284-0b9b-4876-b680-4ee0d6ee0ed7/1a990e4c-7950-4fbe-9b2e-533f3df9e505"
+					(reference "C808")
+					(unit 1)
+				)
+				(path "/6e74608c-23b9-4b98-8fc4-fa8fd655ae50/343e6ab8-61bf-4409-bd59-a9fdebf952af/1a990e4c-7950-4fbe-9b2e-533f3df9e505"
+					(reference "C1303")
+					(unit 1)
+				)
+			)
+		)
+	)
+	(symbol
+		(lib_id "Device:C")
 		(at 200.66 129.54 0)
 		(unit 1)
@@
 			)
 		)
-		(property "Value" "4,7u"
+		(property "Value" "27n"
 			(at 204.47 130.8099 0)
 			(show_name no)
@@
 			)
 		)
-		(property "Value" "4,7u"
+		(property "Value" "100n"
 			(at 204.47 110.4899 0)
 			(show_name no)
