File: hardware_main/Linear_PostReg.kicad_sch (KiCad schematic)
At the start: 52 parts, among them Q301 BCP56, Q302 BSS138, Q303 TIP125, Q304 BCP56, U301 TLV4387PWR, U302 LMV331

Commit message: routing
Parts:
- R306, R309: value 4,3k -> 2,2k
- R313, R314: value 62k -> 33k
- R316: value 18k -> 11k
- R317: value 1,6k -> 1k
Other:
- note added: "G=1/15 Vin=36V --> Vout=2,4V"
- note added: "G=12 Vin=200mV --> Vout=2,4V"
- note removed: "G=0,06935 Vin=36V --> Vout=2,49677V"
- note removed: "G=12,25 Vin=200mV --> Vout=2,45V"
Changed lines of the file:
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@@
 		)
 	)
-	(text "G=0,06935\nVin=36V --> Vout=2,49677V"
+	(text "G=1/15\nVin=36V --> Vout=2,4V"
 		(exclude_from_sim no)
 		(at 95.25 137.16 0)
@@
 	(text "~12mA"
 		(exclude_from_sim no)
-		(at 266.7 133.35 0)
+		(at 266.7 124.46 0)
 		(effects
 			(font
@@
 		)
 	)
-	(text "G=12,25\nVin=200mV --> Vout=2,45V\n"
+	(text "G=12\nVin=200mV --> Vout=2,4V\n"
 		(exclude_from_sim no)
 		(at 149.86 99.06 0)
@@
 			)
 		)
-		(property "Value" "62k"
+		(property "Value" "33k"
 			(at 167.64 143.51 90)
 			(show_name no)
@@
 			)
 		)
-		(property "Value" "4,3k"
+		(property "Value" "2,2k"
 			(at 132.08 152.4 90)
 			(show_name no)
@@
 			)
 		)
-		(property "Value" "18k"
+		(property "Value" "11k"
 			(at 175.26 110.4899 0)
 			(show_name no)
@@
 			)
 		)
-		(property "Value" "62k"
+		(property "Value" "33k"
 			(at 167.64 138.43 90)
 			(show_name no)
@@
 			)
 		)
-		(property "Value" "4,3k"
+		(property "Value" "2,2k"
 			(at 144.78 133.3499 0)
 			(show_name no)
@@
 			)
 		)
-		(property "Value" "1,6k"
+		(property "Value" "1k"
 			(at 175.26 120.6499 0)
 			(show_name no)
