File: hardware_main/Linear_PostReg.kicad_sch (KiCad schematic)
At the start: 52 parts, among them Q301 BCP56, Q302 BSS138, Q303 TIP125, Q304 BCP56, U301 TLV4387PWR, U302 LMV331

Commit message: stability calc
Parts:
- C1014: value 100p -> 22p; now fitted
- C303: value 1n -> 47n
- C304: value 100p -> 27n
- R303: value 1k -> 18k
- R306, R309: value 2,2k -> 2,2k 0,1%
- R313, R314: value 33k -> 33k 0,1%
- R316: value 11k -> 11k 0,1%
- R317: value 1k -> 1k 0,1%
Other:
- moved on the sheet: C306
Changed lines of the file:
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@@
 	)
 	(junction
+		(at 157.48 138.43)
+		(diameter 0)
+		(color 0 0 0 0)
+	)
+	(junction
 		(at 109.22 46.99)
 		(diameter 0)
@@
 	)
 	(junction
-		(at 152.4 138.43)
-		(diameter 0)
-		(color 0 0 0 0)
-	)
-	(junction
 		(at 171.45 43.18)
 		(diameter 0)
@@
 	(wire
 		(pts
-			(xy 142.24 138.43) (xy 152.4 138.43)
+			(xy 142.24 138.43) (xy 157.48 138.43)
 		)
 		(stroke
@@
 	(wire
 		(pts
-			(xy 152.4 135.89) (xy 152.4 138.43)
+			(xy 157.48 135.89) (xy 157.48 138.43)
 		)
 		(stroke
@@
 	(wire
 		(pts
-			(xy 152.4 124.46) (xy 152.4 128.27)
+			(xy 157.48 124.46) (xy 157.48 128.27)
 		)
 		(stroke
@@
 	(wire
 		(pts
-			(xy 152.4 138.43) (xy 163.83 138.43)
-		)
-		(stroke
-			(width 0)
-			(type default)
-		)
-	)
-	(wire
-		(pts
 			(xy 81.28 78.74) (xy 81.28 71.12)
 		)
@@
 	(wire
 		(pts
-			(xy 152.4 124.46) (xy 142.24 124.46)
+			(xy 157.48 124.46) (xy 142.24 124.46)
 		)
 		(stroke
@@
 	(wire
 		(pts
+			(xy 157.48 138.43) (xy 163.83 138.43)
+		)
+		(stroke
+			(width 0)
+			(type default)
+		)
+	)
+	(wire
+		(pts
 			(xy 161.29 105.41) (xy 161.29 102.87)
 		)
@@
 		(dnp no)
 		(property "Reference" "R314"
-			(at 167.64 140.97 90)
+			(at 170.18 146.05 90)
 			(show_name no)
 			(do_not_autoplace no)
@@
 			)
 		)
-		(property "Value" "33k"
-			(at 167.64 143.51 90)
+		(property "Value" "33k 0,1%"
+			(at 170.18 148.59 90)
 			(show_name no)
 			(do_not_autoplace no)
@@
 			)
 		)
-		(property "Value" "1k"
+		(property "Value" "18k"
 			(at 101.6 39.37 90)
 			(show_name no)
@@
 			)
 		)
-		(property "Value" "1n"
+		(property "Value" "47n"
 			(at 93.98 38.1 90)
 			(show_name no)
@@
 		(dnp no)
 		(property "Reference" "R306"
-			(at 132.08 149.86 90)
+			(at 132.08 147.32 90)
 			(show_name no)
 			(do_not_autoplace no)
@@
 			)
 		)
-		(property "Value" "2,2k"
-			(at 132.08 152.4 90)
+		(property "Value" "2,2k 0,1%"
+			(at 132.08 149.86 90)
 			(show_name no)
 			(do_not_autoplace no)
@@
 			)
 		)
-		(property "Value" "11k"
+		(property "Value" "11k 0,1%"
 			(at 175.26 110.4899 0)
 			(show_name no)
@@
 		(on_board yes)
 		(in_pos_files yes)
-		(dnp yes)
+		(dnp no)
 		(property "Reference" "C1014"
 			(at 97.79 43.18 90)
@@
 			)
 		)
-		(property "Value" "100p"
+		(property "Value" "22p"
 			(at 97.79 45.72 90)
 			(show_name no)
@@
 	(symbol
 		(lib_id "Device:C")
-		(at 152.4 132.08 0)
+		(at 157.48 132.08 0)
 		(unit 1)
 		(body_style 1)
@@
 		(fields_autoplaced yes)
 		(property "Reference" "C306"
-			(at 156.21 130.8099 0)
+			(at 161.29 130.8099 0)
 			(show_name no)
 			(do_not_autoplace no)
@@
 		)
 		(property "Value" "10p"
-			(at 156.21 133.3499 0)
+			(at 161.29 133.3499 0)
 			(show_name no)
 			(do_not_autoplace no)
@@
 		)
 		(property "Footprint" "Capacitor_SMD:C_0603_1608Metric"
-			(at 153.3652 135.89 0)
+			(at 158.4452 135.89 0)
 			(hide yes)
 			(show_name no)
@@
 		)
 		(property "Datasheet" ""
-			(at 152.4 132.08 0)
+			(at 157.48 132.08 0)
 			(hide yes)
 			(show_name no)
@@
 		)
 		(property "Description" "Unpolarized capacitor"
-			(at 152.4 132.08 0)
+			(at 157.48 132.08 0)
 			(hide yes)
 			(show_name no)
@@
 		(dnp no)
 		(property "Reference" "R313"
-			(at 167.64 135.89 90)
+			(at 170.18 133.35 90)
 			(show_name no)
 			(do_not_autoplace no)
@@
 			)
 		)
-		(property "Value" "33k"
-			(at 167.64 138.43 90)
+		(property "Value" "33k 0,1%"
+			(at 170.18 135.89 90)
 			(show_name no)
 			(do_not_autoplace no)
@@
 			)
 		)
-		(property "Value" "2,2k"
+		(property "Value" "2,2k 0,1%"
 			(at 144.78 133.3499 0)
 			(show_name no)
@@
 			)
 		)
-		(property "Value" "100p"
+		(property "Value" "27n"
 			(at 93.98 77.47 90)
 			(show_name no)
@@
 			)
 		)
-		(property "Value" "1k"
+		(property "Value" "1k 0,1%"
 			(at 175.26 120.6499 0)
 			(show_name no)

Commit message: calc and cleanup
Parts:
- added C1015: 100n, Capacitor_SMD:C_0603_1608Metric, symbol Device:C
- F301: value Fuse -> 3A
Connections:
- net +3V3: now also C1015.1
- net GND: now also C1015.2
Changed lines of the file:
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@@
 	)
 	(junction
+		(at 128.27 102.87)
+		(diameter 0)
+		(color 0 0 0 0)
+	)
+	(junction
 		(at 157.48 21.59)
 		(diameter 0)
@@
 	)
 	(junction
-		(at 128.27 102.87)
-		(diameter 0)
-		(color 0 0 0 0)
-	)
-	(junction
 		(at 109.22 68.58)
 		(diameter 0)
@@
 	(wire
 		(pts
+			(xy 80.01 187.96) (xy 80.01 182.88)
+		)
+		(stroke
+			(width 0)
+			(type default)
+		)
+	)
+	(wire
+		(pts
 			(xy 172.72 102.87) (xy 177.8 102.87)
 		)
@@
 	(wire
 		(pts
+			(xy 80.01 170.18) (xy 80.01 175.26)
+		)
+		(stroke
+			(width 0)
+			(type default)
+		)
+	)
+	(wire
+		(pts
 			(xy 22.86 165.1) (xy 22.86 171.45)
 		)
@@
 		)
 	)
+	(label "+3V3"
+		(at 80.01 170.18 270)
+		(effects
+			(font
+				(size 1.27 1.27)
+			)
+			(justify right bottom)
+		)
+	)
 	(label "-1V2"
 		(at 156.21 193.04 90)
@@
 		)
 	)
+	(label "GND"
+		(at 80.01 187.96 90)
+		(effects
+			(font
+				(size 1.27 1.27)
+			)
+			(justify left bottom)
+		)
+	)
 	(label "OUT+"
 		(at 176.53 138.43 0)
@@
 			)
 		)
-		(property "Value" "Fuse"
+		(property "Value" "3A"
 			(at 220.98 54.61 90)
 			(show_name no)
@@
 					(unit 1)
 				)
+			)
+		)
+	)
+	(symbol
+		(lib_id "Device:C")
+		(at 80.01 179.07 0)
+		(unit 1)
+		(body_style 1)
+		(exclude_from_sim no)
+		(in_bom yes)
+		(on_board yes)
+		(in_pos_files yes)
+		(dnp no)
+		(fields_autoplaced yes)
+		(property "Reference" "C1015"
+			(at 83.82 177.7999 0)
+			(show_name no)
+			(do_not_autoplace no)
+			(effects
+				(font
+					(size 1.27 1.27)
+				)
+				(justify left)
+			)
+		)
+		(property "Value" "100n"
+			(at 83.82 180.3399 0)
+			(show_name no)
+			(do_not_autoplace no)
+			(effects
+				(font
+					(size 1.27 1.27)
+				)
+				(justify left)
+			)
+		)
+		(property "Footprint" "Capacitor_SMD:C_0603_1608Metric"
+			(at 80.9752 182.88 0)
+			(hide yes)
+			(show_name no)
+			(do_not_autoplace no)
+			(effects
+				(font
+					(size 1.27 1.27)
+				)
+			)
+		)
+		(property "Datasheet" ""
+			(at 80.01 179.07 0)
+			(hide yes)
+			(show_name no)
+			(do_not_autoplace no)
+			(effects
+				(font
+					(size 1.27 1.27)
+				)
+			)
+		)
+		(property "Description" "Unpolarized capacitor"
+			(at 80.01 179.07 0)
+			(hide yes)
+			(show_name no)
+			(do_not_autoplace no)
+			(effects
+				(font
+					(size 1.27 1.27)
+				)
+			)
+		)
+		(pin "1"
+		)
+		(pin "2"
+		)
+		(instances
+			(project "DualPreRegPowerSupply"
+				(path "/6e74608c-23b9-4b98-8fc4-fa8fd655ae50/19bfe284-0b9b-4876-b680-4ee0d6ee0ed7/f35a5384-6f7b-4a9d-a7fe-0a11cd4efe3d"
+					(reference "C1015")
+					(unit 1)
+				)
+				(path "/6e74608c-23b9-4b98-8fc4-fa8fd655ae50/343e6ab8-61bf-4409-bd59-a9fdebf952af/f35a5384-6f7b-4a9d-a7fe-0a11cd4efe3d"
+					(reference "C1205")
+					(unit 1)
+				)
