File: hardware_main/DualPreRegPowerSupply.kicad_sch (KiCad schematic)
At the start: 4 parts

Commit message: routing
Changed lines of the file:
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@@
 	(sheet
 		(at 160.02 59.69)
-		(size 53.34 22.86)
+		(size 55.88 22.86)
 		(exclude_from_sim no)
 		(in_bom yes)
@@
 	(sheet
 		(at 160.02 97.79)
-		(size 53.34 22.86)
+		(size 55.88 22.86)
 		(exclude_from_sim no)
 		(in_bom yes)
