File: hardware_main/Control.kicad_sch (KiCad schematic)
At the start: 16 parts, among them J203 Conn_02x04_Odd_Even, J204 Conn_02x05_Odd_Even, J205 Conn_01x04_Pin, M401 Fan_4pin, U401 TMP1075D

Commit message: routing
Other:
- moved on the sheet: C404
Changed lines of the file:
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@@
 	(wire
 		(pts
-			(xy 220.98 21.59) (xy 220.98 22.86)
+			(xy 144.78 69.85) (xy 130.81 69.85)
 		)
 		(stroke
@@
 	(wire
 		(pts
-			(xy 144.78 69.85) (xy 130.81 69.85)
+			(xy 220.98 134.62) (xy 234.95 134.62)
 		)
 		(stroke
@@
 	(wire
 		(pts
-			(xy 220.98 134.62) (xy 234.95 134.62)
+			(xy 220.98 20.32) (xy 220.98 22.86)
 		)
 		(stroke
@@
 	(wire
 		(pts
-			(xy 220.98 35.56) (xy 220.98 36.83)
+			(xy 220.98 35.56) (xy 220.98 38.1)
 		)
 		(stroke
@@
 	(symbol
 		(lib_id "Device:C")
-		(at 238.76 29.21 0)
+		(at 220.98 59.69 0)
 		(unit 1)
 		(body_style 1)
@@
 		(dnp no)
 		(property "Reference" "C404"
-			(at 241.3 27.94 0)
+			(at 223.52 58.42 0)
 			(show_name no)
 			(do_not_autoplace no)
@@
 		)
 		(property "Value" "10u"
-			(at 241.3 30.48 0)
+			(at 223.52 60.96 0)
 			(show_name no)
 			(do_not_autoplace no)
@@
 		)
 		(property "Footprint" "Capacitor_SMD:C_0805_2012Metric"
-			(at 239.7252 33.02 0)
+			(at 221.9452 63.5 0)
 			(hide yes)
 			(show_name no)
@@
 		)
 		(property "Datasheet" ""
-			(at 238.76 29.21 0)
+			(at 220.98 59.69 0)
 			(hide yes)
 			(show_name no)
@@
 		)
 		(property "Description" "Unpolarized capacitor"
-			(at 238.76 29.21 0)
+			(at 220.98 59.69 0)
 			(hide yes)
 			(show_name no)
@@
 	(symbol
 		(lib_id "power:GNDD")
-		(at 220.98 36.83 0)
+		(at 220.98 38.1 0)
 		(unit 1)
 		(body_style 1)
@@
 		(fields_autoplaced yes)
 		(property "Reference" "#PWR0414"
-			(at 220.98 43.18 0)
+			(at 220.98 44.45 0)
 			(hide yes)
 			(show_name no)
@@
 		)
 		(property "Value" "GNDD"
-			(at 220.98 40.64 0)
+			(at 220.98 41.91 0)
 			(show_name no)
 			(do_not_autoplace no)
@@
 		)
 		(property "Footprint" ""
-			(at 220.98 36.83 0)
+			(at 220.98 38.1 0)
 			(hide yes)
 			(show_name no)
@@
 		)
 		(property "Datasheet" ""
-			(at 220.98 36.83 0)
+			(at 220.98 38.1 0)
 			(hide yes)
 			(show_name no)
@@
 		)
 		(property "Description" "Power symbol creates a global label with name \"GNDD\" , digital ground"
-			(at 220.98 36.83 0)
+			(at 220.98 38.1 0)
 			(hide yes)
 			(show_name no)
@@
 	(symbol
 		(lib_id "power:GNDD")
-		(at 238.76 33.02 0)
+		(at 220.98 63.5 0)
 		(unit 1)
 		(body_style 1)
@@
 		(fields_autoplaced yes)
 		(property "Reference" "#PWR0420"
-			(at 238.76 39.37 0)
+			(at 220.98 69.85 0)
 			(hide yes)
 			(show_name no)
@@
 		)
 		(property "Value" "GNDD"
-			(at 238.76 36.83 0)
+			(at 220.98 67.31 0)
 			(show_name no)
 			(do_not_autoplace no)
@@
 		)
 		(property "Footprint" ""
-			(at 238.76 33.02 0)
+			(at 220.98 63.5 0)
 			(hide yes)
 			(show_name no)
@@
 		)
 		(property "Datasheet" ""
-			(at 238.76 33.02 0)
+			(at 220.98 63.5 0)
 			(hide yes)
 			(show_name no)
@@
 		)
 		(property "Description" "Power symbol creates a global label with name \"GNDD\" , digital ground"
-			(at 238.76 33.02 0)
+			(at 220.98 63.5 0)
 			(hide yes)
 			(show_name no)
@@
 	(symbol
 		(lib_id "power:+12V")
-		(at 220.98 21.59 0)
+		(at 220.98 20.32 0)
 		(unit 1)
 		(body_style 1)
@@
 		(fields_autoplaced yes)
 		(property "Reference" "#PWR0413"
-			(at 220.98 25.4 0)
+			(at 220.98 24.13 0)
 			(hide yes)
 			(show_name no)
@@
 		)
 		(property "Value" "+12V"
-			(at 220.98 16.51 0)
+			(at 220.98 15.24 0)
 			(show_name no)
 			(do_not_autoplace no)
@@
 		)
 		(property "Footprint" ""
-			(at 220.98 21.59 0)
+			(at 220.98 20.32 0)
 			(hide yes)
 			(show_name no)
@@
 		)
 		(property "Datasheet" ""
-			(at 220.98 21.59 0)
+			(at 220.98 20.32 0)
 			(hide yes)
 			(show_name no)
@@
 		)
 		(property "Description" "Power symbol creates a global label with name \"+12V\""
-			(at 220.98 21.59 0)
+			(at 220.98 20.32 0)
 			(hide yes)
 			(show_name no)
@@
 	(symbol
 		(lib_id "power:+12V")
-		(at 238.76 25.4 0)
+		(at 220.98 55.88 0)
 		(unit 1)
 		(body_style 1)
@@
 		(fields_autoplaced yes)
 		(property "Reference" "#PWR0419"
-			(at 238.76 29.21 0)
+			(at 220.98 59.69 0)
 			(hide yes)
 			(show_name no)
@@
 		)
 		(property "Value" "+12V"
-			(at 238.76 20.32 0)
+			(at 220.98 50.8 0)
 			(show_name no)
 			(do_not_autoplace no)
@@
 		)
 		(property "Footprint" ""
-			(at 238.76 25.4 0)
+			(at 220.98 55.88 0)
 			(hide yes)
 			(show_name no)
@@
 		)
 		(property "Datasheet" ""
-			(at 238.76 25.4 0)
+			(at 220.98 55.88 0)
 			(hide yes)
 			(show_name no)
@@
 		)
 		(property "Description" "Power symbol creates a global label with name \"+12V\""
-			(at 238.76 25.4 0)
+			(at 220.98 55.88 0)
 			(hide yes)
 			(show_name no)

Commit message: routing
Parts:
- R201, R203: value 2k -> 10k
Connections:
- net W5500_CS: now also A401.17 (GPIO17), J204.1 (Pin_1); no longer A401.20 (GPIO20), J204.7 (Pin_7)
- net W5500_MISO: now also A401.20 (GPIO20), J204.7 (Pin_7); no longer A401.16 (GPIO16/LED), J204.1 (Pin_1)
- net Buzzer: no longer names the net of A401.27 (GPIO27_ADC1)

Commit message: routing
Parts:
- removed C401: 100n, Capacitor_SMD:C_0603_1608Metric, symbol Device:C
- removed R401, R402: 2k, Resistor_SMD:R_0603_1608Metric, symbol Device:R
- removed U401: TMP1075D, Package_SO:SO-8_3.9x4.9mm_P1.27mm, symbol Sensor_Temperature:TMP1075D
- added C203: 1u, Capacitor_SMD:C_0603_1608Metric, symbol Device:C
- added R204, R205: 10k, Resistor_SMD:R_0603_1608Metric, symbol Device:R
- added TH201: Thermistor_NTC, LibEigen:Flex NTC, symbol Device:Thermistor_NTC
Connections:
- net +3.3V: now also R204.2
- net GNDD: now also C203.2, TH201.2
- net at A401.29 (GPIO29_ADC3): now also C203.1, R205.2
- new net: R204.1, R205.1, TH201.1
Other:
- note removed: "1001111"
