File: hardware_main/DCDCTracking.kicad_sch (KiCad schematic)
At the start: 29 parts, among them Q501 MMBT3906, U501 LT8612

Commit message: routing
Other:
- note removed: "Delta I (5Vout) = 0,62 A Delta I (30Vout) = 0,73 A"
Changed lines of the file:
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@@
-		)
-	)
-	(text "Delta I (5Vout) = 0,62 A\nDelta I (30Vout) = 0,73 A"
-		(exclude_from_sim no)
-		(at 146.05 60.96 0)
-		(effects
-			(font
-				(size 1.27 1.27)
-			)
-			(justify left top)
 		)
 	)

Commit message: routing
Parts:
- R504: now not fitted
Changed lines of the file:
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@@
 		(on_board yes)
 		(in_pos_files yes)
-		(dnp no)
+		(dnp yes)
 		(property "Reference" "R504"
 			(at 127 76.2 90)

Commit message: routing
Parts:
- removed R504: 49,9k, Resistor_SMD:R_0603_1608Metric, symbol Device:R
- added D904: green LED PG, LED_SMD:LED_0603_1608Metric, symbol Device:LED
- added Q901: BSS138, Package_TO_SOT_SMD:SOT-23, symbol Transistor_FET:BSS138
- added R905: 2,4k, Resistor_SMD:R_0603_1608Metric, symbol Device:R
- added R906: 10k, Resistor_SMD:R_0603_1608Metric, symbol Device:R
- added TP901: TestPoint_Alt, TestPoint:TestPoint_Pad_D1.0mm, symbol Connector:TestPoint_Alt
Connections:
- net +3V3: now also D904.2 (A), R906.1
- net GND: now also Q901.2 (S)
- net PG: now reaches U501.23 (PG)
- net PG: now also Q901.1 (G), R906.2, TP901.1
- new net: D904.1 (K), R905.1
- new net: Q901.3 (D), R905.2
Other:
- moved on the sheet: C501, C502, C503, C504, C505, C506, C507, C508, C509, C510, C511, C512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
