File: hardware_main/DCDCTracking.kicad_sch (KiCad schematic)
At the start: 33 parts, among them Q501 MMBT3906, Q901 BSS138, U501 LT8612

Commit message: stability calc
Parts:
- added C908: opt, Capacitor_SMD:C_0603_1608Metric, symbol Device:C
Connections:
- net GND: now also C908.2
- net at C510.2, Q501.1 (B), R508.1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: now also C908.1
Changed lines of the file:
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@@
+	)
+	(junction
+		(at 204.47 137.16)
+		(diameter 0)
+		(color 0 0 0 0)
 	)
 	(junction
@@
 	)
 	(junction
+		(at 204.47 109.22)
+		(diameter 0)
+		(color 0 0 0 0)
+	)
+	(junction
 		(at 222.25 73.66)
 		(diameter 0)
@@
 	(wire
 		(pts
+			(xy 204.47 128.27) (xy 204.47 137.16)
+		)
+		(stroke
+			(width 0)
+			(type default)
+		)
+	)
+	(wire
+		(pts
 			(xy 193.04 115.57) (xy 193.04 116.84)
 		)
@@
 	(wire
 		(pts
-			(xy 193.04 137.16) (xy 237.49 137.16)
+			(xy 193.04 137.16) (xy 204.47 137.16)
 		)
 		(stroke
@@
 	(wire
 		(pts
+			(xy 204.47 109.22) (xy 204.47 120.65)
+		)
+		(stroke
+			(width 0)
+			(type default)
+		)
+	)
+	(wire
+		(pts
 			(xy 137.16 95.25) (xy 137.16 96.52)
 		)
@@
 	(wire
 		(pts
+			(xy 204.47 137.16) (xy 237.49 137.16)
+		)
+		(stroke
+			(width 0)
+			(type default)
+		)
+	)
+	(wire
+		(pts
 			(xy 227.33 109.22) (xy 245.11 109.22)
 		)
@@
 	(wire
 		(pts
+			(xy 204.47 109.22) (xy 217.17 109.22)
+		)
+		(stroke
+			(width 0)
+			(type default)
+		)
+	)
+	(wire
+		(pts
 			(xy 62.23 63.5) (xy 74.93 63.5)
 		)
@@
 	(wire
 		(pts
-			(xy 203.2 109.22) (xy 217.17 109.22)
+			(xy 203.2 109.22) (xy 204.47 109.22)
 		)
 		(stroke
@@
 					(unit 1)
 				)
+			)
+		)
+	)
+	(symbol
+		(lib_id "Device:C")
+		(at 204.47 124.46 0)
+		(unit 1)
+		(body_style 1)
+		(exclude_from_sim no)
+		(in_bom yes)
+		(on_board yes)
+		(in_pos_files yes)
+		(dnp yes)
+		(fields_autoplaced yes)
+		(property "Reference" "C908"
+			(at 208.28 123.1899 0)
+			(show_name no)
+			(do_not_autoplace no)
+			(effects
+				(font
+					(size 1.27 1.27)
+				)
+				(justify left)
+			)
+		)
+		(property "Value" "opt"
+			(at 208.28 125.7299 0)
+			(show_name no)
+			(do_not_autoplace no)
+			(effects
+				(font
+					(size 1.27 1.27)
+				)
+				(justify left)
+			)
+		)
+		(property "Footprint" "Capacitor_SMD:C_0603_1608Metric"
+			(at 205.4352 128.27 0)
+			(hide yes)
+			(show_name no)
+			(do_not_autoplace no)
+			(effects
+				(font
+					(size 1.27 1.27)
+				)
+			)
+		)
+		(property "Datasheet" ""
+			(at 204.47 124.46 0)
+			(hide yes)
+			(show_name no)
+			(do_not_autoplace no)
+			(effects
+				(font
+					(size 1.27 1.27)
+				)
+			)
+		)
+		(property "Description" "Unpolarized capacitor"
+			(at 204.47 124.46 0)
+			(hide yes)
+			(show_name no)
+			(do_not_autoplace no)
+			(effects
+				(font
+					(size 1.27 1.27)
+				)
+			)
+		)
+		(pin "1"
+		)
+		(pin "2"
+		)
+		(instances
+			(project "DualPreRegPowerSupply"
+				(path "/6e74608c-23b9-4b98-8fc4-fa8fd655ae50/19bfe284-0b9b-4876-b680-4ee0d6ee0ed7/5421e415-5d68-4eaa-8c24-bcc4d6156d8b"
+					(reference "C908")
+					(unit 1)
+				)
+				(path "/6e74608c-23b9-4b98-8fc4-fa8fd655ae50/343e6ab8-61bf-4409-bd59-a9fdebf952af/5421e415-5d68-4eaa-8c24-bcc4d6156d8b"
+					(reference "C1401")
+					(unit 1)
+				)
