File: hardware_main/Digi_Power.kicad_sch (KiCad schematic)
At the start: 18 parts, among them J901 Power Input, U901 AP63200WU

Commit message: routing
Parts:
- added TP306, TP307, TP308: TestPoint_Alt, TestPoint:TestPoint_Keystone_5005-5009_Compact, symbol Connector:TestPoint_Alt
Connections:
- net +12V: now also TP308.1
- net +3.3V: now also TP307.1
- net GNDD: now also TP306.1

Commit message: routing
Parts:
- D902: value LED 12V -> green LED 12V
- D903: value LED 3V3 -> green LED 3V3
Changed lines of the file:
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@@
 			)
 		)
-		(property "Value" "LED 3V3"
+		(property "Value" "green LED 3V3"
 			(at 222.25 38.4174 90)
 			(show_name no)
@@
 		(in_pos_files yes)
 		(dnp no)
-		(fields_autoplaced yes)
 		(property "Reference" "D902"
 			(at 83.82 37.1474 90)
@@
 			)
 		)
-		(property "Value" "LED 12V"
-			(at 83.82 39.6874 90)
-			(show_name no)
-			(do_not_autoplace no)
+		(property "Value" "green LED 12V"
+			(at 83.82 39.37 90)
+			(show_name no)
+			(do_not_autoplace no)
