File: hardware_main/Digi_Power.kicad_sch (KiCad schematic)
At the start: 21 parts, among them J901 Power Input, U901 AP63200WU

Commit message: while build
Parts:
- R904: value ### -> 2,4k
Changed lines of the file:
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@@
 			)
 		)
-		(property "Value" "###"
+		(property "Value" "2,4k"
 			(at 220.98 27.9399 0)
 			(show_name no)
