File: hardware_main/DualPreRegPowerSupply.kicad_pcb (KiCad board)
At the start: 4 copper layers, 100 x 100 mm, 354 parts, among them J101 Power Input, J102 Conn_01x03_Pin, J103 Conn_02x02_Odd_Even, J201 Banana_Red, J202 Banana_Black, J203 Conn_02x04_Odd_Even, J204 Conn_02x05_Odd_Even, J205 Conn_01x04_Pin, J402 Banana_Red, J403 Banana_Black, J601 Power Input, J801 Conn_01x03_Pin, J802 Conn_02x02_Odd_Even, J901 Power Input, M401 Fan_4pin, Q101 MMBT3906, Q102 BCP56, Q103 BSS138, Q104 TIP125, Q105 BSS138, Q106 BSS138, Q107 BCP56, Q301 BCP56, Q302 BSS138, Q303 TIP125, Q304 BCP56, Q501 MMBT3906, Q801 BSS138, Q802 BSS138, U1002 AP7383, U1003 LM2776, U1004 XC6901D121MR-G, U101 TLV4387PWR, U102 ISO6721RFBD, U104 LT8612, U105 LMV331, U106 ATtiny1614-SS, U107 ADS1118IDGS, U108 MCP48FVB22, U109 AP7383, U110 LM2776, U111 XC6901D121MR-G, U1501 LMR51606, U301 TLV4387PWR, U302 LMV331, U401 TMP1075D, U501 LT8612, U601 LMR51606, U701 ADS1118IDGS, U702 MCP48FVB22, U801 ISO6721RFBD, U802 ATtiny1614-SS, U901 AP63200WU

Commit message: routing
Parts:
- added TP306: TestPoint_Alt, TestPoint:TestPoint_Keystone_5005-5009_Compact, B.Cu at (159.6, 67.8)
- added TP307: TestPoint_Alt, TestPoint:TestPoint_Keystone_5005-5009_Compact, B.Cu at (154.3, 67.8)
- added TP308: TestPoint_Alt, TestPoint:TestPoint_Keystone_5005-5009_Compact, B.Cu at (151.8, 55.7)
- C113, C114, C701, C702: value ## -> 4,7u
- D101, D601: value SM6T36A -> SMBJ40A
- D201, D401: value SM6T36A -> SMBJ36A
- M401: moved to B.Cu
- R104, R105, R701, R702: value ## -> 1k
- R116, R119, R306, R309: value 4,3k -> 2,2k
- R127, R128, R313, R314: value 62k -> 33k
- R131, R316: value 18k -> 11k
- R132, R317: value 1,6k -> 1k
- moved R202 7.24 mm to (159.7, 59.2), turned to 0 degrees
- moved M401 7.20 mm to (158.3, 49.8), turned to 180 degrees
- moved C404 5.52 mm to (157.0, 54.8), turned to 0 degrees
- moved R404 5.28 mm to (159.7, 57.6), turned to 180 degrees
- moved D903 2.88 mm to (155.3, 62.4)
- moved R904 2.88 mm to (155.3, 59.3)
- moved D902 2.51 mm to (153.4, 62.4)
- moved R901 2.51 mm to (153.4, 59.3)
Routing:
- net Net-(M401-PWM): track 2.30 -> 12.5 mm
- net /Control/FanPWM: track 65.4 -> 58.7 mm
- net +12V: track 26.6 -> 31.2 mm
- net GNDD: track 29.6 -> 32.4 mm
- added copper zone on F.Cu, net GND_Ch2
Other:
- board text added: "-12V+"
- board text added: "-40V+"
- board text added: "Ch2"

Commit message: routing
Connections:
- A401 pad 16: /Control/W5500_MISO -> unconnected-(A401-GPIO16/LED-Pad16)
- A401 pad 17: unconnected-(A401-GPIO17-Pad17) -> /Control/W5500_CS
- A401 pad 20: /Control/W5500_CS -> /Control/W5500_MISO
- A401 pad 27: /Control/Buzzer -> unconnected-(A401-GPIO27_ADC1-Pad27)
- J204 pad 1: /Control/W5500_MISO -> /Control/W5500_CS
- J204 pad 7: /Control/W5500_CS -> /Control/W5500_MISO
Routing:
- net /Control/W5500_MISO: track 33.0 -> 40.3 mm
- net /Control/W5500_CS: track 40.3 -> 34.8 mm
- net /Ch1Power/DCDCTracking/DCDC_FB: track 26.7 -> 25.1 mm
Other:
- board size 100 x 100 mm -> 99.6 x 100 mm

Commit message: routing
Parts:
- removed C401: 100n, Capacitor_SMD:C_0603_1608Metric
- removed R111, R504: 49,9k, Resistor_SMD:R_0603_1608Metric
- removed R401, R402: 2k, Resistor_SMD:R_0603_1608Metric
- removed U401: TMP1075D, Package_SO:SO-8_3.9x4.9mm_P1.27mm
- added C203: 1u, Capacitor_SMD:C_0603_1608Metric, B.Cu at (161.3, 106.0)
- added D1401: green LED PG, LED_SMD:LED_0603_1608Metric, B.Cu at (171.6, 61.5)
- added D904: green LED PG, LED_SMD:LED_0603_1608Metric, B.Cu at (112.4, 63.0)
- added Q1401: BSS138, Package_TO_SOT_SMD:SOT-23, B.Cu at (165.1, 62.8)
- added Q901: BSS138, Package_TO_SOT_SMD:SOT-23, B.Cu at (108.2, 63.2)
- added R1401: 2,4k, Resistor_SMD:R_0603_1608Metric, B.Cu at (168.4, 61.5)
- added R1402: 10k, Resistor_SMD:R_0603_1608Metric, B.Cu at (168.3, 63.1)
- added R204: 10k, Resistor_SMD:R_0603_1608Metric, B.Cu at (151.1, 90.0)
- added R205: 10k, Resistor_SMD:R_0603_1608Metric, B.Cu at (149.0, 90.0)
- added R905: 2,4k, Resistor_SMD:R_0603_1608Metric, B.Cu at (110.8, 63.0)
- added R906: 10k, Resistor_SMD:R_0603_1608Metric, B.Cu at (107.5, 66.0)
- added TH201: Thermistor_NTC, LibEigen:Flex NTC, F.Cu at (150.0, 90.0)
- added TP1401: TestPoint_Alt, TestPoint:TestPoint_Pad_D1.0mm, B.Cu at (164.3, 59.5)
- added TP901: TestPoint_Alt, TestPoint:TestPoint_Pad_D1.0mm, B.Cu at (108.1, 67.8)
- D1001, D105, D903: value LED 3V3 -> green LED 3V3
- D1002, D106: value LED -5V -> green LED -5V
- D103, D107, D801, D802: value LED 3V3 -> red LED 3V3
- D104, D602: value LED 40V -> green LED 40V
- D902: value LED 12V -> green LED 12V
- R201, R203: value 2k -> 10k
- moved TP608 10.2 mm to (117.6, 59.5)
- moved TP606 6.15 mm to (102.5, 81.1)
- moved R1003 5.78 mm to (101.2, 59.7), turned to -90 degrees
- moved TP603 5.20 mm to (102.8, 72.4)
- moved C110 4.40 mm to (175.9, 60.2), turned to 0 degrees
- moved D602 4.08 mm to (105.0, 62.8), turned to 90 degrees
- moved R1004 2.73 mm to (103.1, 59.7), turned to -90 degrees
- moved D1002 1.94 mm to (103.1, 62.8), turned to 90 degrees
- moved D1001 1.45 mm to (101.2, 62.8), turned to 90 degrees
- moved R601 0.50 mm to (105.0, 59.7), turned to -90 degrees
Connections:
- A401 pad 29: unconnected-(A401-GPIO29_ADC3-Pad29) -> Net-(A401-GPIO29_ADC3)
- U104 pad 23: Net-(U104-PG) -> /Ch1Power1/DCDCTracking/PG
- U501 pad 23: Net-(U501-PG) -> /Ch1Power/DCDCTracking/PG
Routing:
- net /Control/SCL: track 60.4 -> 24.1 mm
- net /Control/SDA: track 57.8 -> 25.2 mm
- net Net-(A401-GPIO29_ADC3): track 0.00 -> 22.5 mm, vias 0 -> 2
- net +3.3V: track 27.4 -> 15.6 mm, vias 19 -> 16
- net /Ch1Power/DCDCTracking/SW_OUT: track 24.8 -> 15.0 mm
- net /Ch1Power1/DCDCTracking/PG: track 0.00 -> 9.71 mm
- net /Ch1Power/DCDCTracking/PG: track 0.00 -> 9.50 mm
- net /Ch1Power1/DCDCTracking/SW_OUT: track 21.0 -> 12.4 mm
- net Net-(Q1401-D): track 0.00 -> 7.19 mm, vias 0 -> 2
- net Net-(R204-Pad1): track 0.00 -> 6.72 mm, vias 0 -> 1
- net GNDD: track 32.4 -> 25.7 mm
- net /Control/W5500_SCLK: track 41.1 -> 37.6 mm
- net Net-(D1002-K): track 21.8 -> 25.2 mm
- net Net-(U501-PG): track 3.15 -> 0.00 mm
- net /Control/W5500_MOSI: track 43.0 -> 40.4 mm
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Other:
- outline, holes or cut-outs redrawn
- board text added: "+3,3V"
- board text added: "+40V"
- board text added: "-1,2V"
- board text added: "CC"
- board text added: "DCDC_PG"
- board text added: "OE"
- board text added: "PG"
