File: hardware_main/DualPreRegPowerSupply.kicad_pcb (KiCad board)
At the start: 4 copper layers, 99.6 x 100 mm, 365 parts, among them J101 Power Input, J102 Conn_01x03_Pin, J103 Conn_02x02_Odd_Even, J201 Banana_Red, J202 Banana_Black, J203 Conn_02x04_Odd_Even, J204 Conn_02x05_Odd_Even, J205 Conn_01x04_Pin, J402 Banana_Red, J403 Banana_Black, J601 Power Input, J801 Conn_01x03_Pin, J802 Conn_02x02_Odd_Even, J901 Power Input, M401 Fan_4pin, Q101 MMBT3906, Q102 BCP56, Q103 BSS138, Q104 TIP125, Q105 BSS138, Q106 BSS138, Q107 BCP56, Q1401 BSS138, Q301 BCP56, Q302 BSS138, Q303 TIP125, Q304 BCP56, Q501 MMBT3906, Q801 BSS138, Q802 BSS138, Q901 BSS138, U1002 AP7383, U1003 LM2776, U1004 XC6901D121MR-G, U101 TLV4387PWR, U102 ISO6721RFBD, U104 LT8612, U105 LMV331, U106 ATtiny1614-SS, U107 ADS1118IDGS, U108 MCP48FVB22, U109 AP7383, U110 LM2776, U111 XC6901D121MR-G, U1501 LMR51606, U301 TLV4387PWR, U302 LMV331, U501 LT8612, U601 LMR51606, U701 ADS1118IDGS, U702 MCP48FVB22, U801 ISO6721RFBD, U802 ATtiny1614-SS, U901 AP63200WU

Commit message: stability calc
Parts:
- added C1301: 4,7u, Capacitor_SMD:C_0603_1608Metric, B.Cu at (197.7, 100.9)
- added C1302: 4,7u, Capacitor_SMD:C_0603_1608Metric, B.Cu at (195.5, 100.9)
- added C1401: opt, Capacitor_SMD:C_0603_1608Metric, B.Cu at (164.6, 76.5)
- added C806: 4,7u, Capacitor_SMD:C_0603_1608Metric, F.Cu at (115.5, 102.1)
- added C807: 4,7u, Capacitor_SMD:C_0603_1608Metric, F.Cu at (113.9, 102.1)
- added C908: opt, Capacitor_SMD:C_0603_1608Metric, B.Cu at (106.8, 84.2)
- added R1301: 1k, Resistor_SMD:R_0603_1608Metric, B.Cu at (197.7, 97.8)
- added R1302: 1k, Resistor_SMD:R_0603_1608Metric, B.Cu at (195.5, 97.8)
- added R807: 1k, Resistor_SMD:R_0603_1608Metric, F.Cu at (117.1, 102.1)
- added R808: 1k, Resistor_SMD:R_0603_1608Metric, F.Cu at (112.3, 102.1)
- C1001, C1002, C105, C107: value 22u -> 10u
- C1014, C1204: value 100p -> 22p
- C111, C303: value 1n -> 47n
- C112, C304: value 100p -> 27n
- C138, C604: value 22u -> 100u
- R106, R303: value 1k -> 18k
- R116, R119, R306, R309: value 2,2k -> 2,2k 0,1%
- R127, R128, R313, R314: value 33k -> 33k 0,1%
- R131, R316: value 11k -> 11k 0,1%
- R132, R317: value 1k -> 1k 0,1%
- moved TP1504 10.8 mm to (198.2, 84.5)
- moved TP1502 0.50 mm to (193.4, 80.4)
- moved TP110 0.31 mm to (164.7, 77.3)
Connections:
- U108 pad 4: /Ch1Power1/DAC_ADC/Vset -> Net-(U108-VA)
- U108 pad 5: /Ch1Power1/DAC_ADC/Iset -> Net-(U108-VB)
- U702 pad 4: /Ch1Power/DAC_ADC/Vset -> Net-(U702-VA)
- U702 pad 5: /Ch1Power/DAC_ADC/Iset -> Net-(U702-VB)
Routing:
- net Net-(U702-VB): track 0.00 -> 7.87 mm, vias 0 -> 1
- net /Ch1Power/DAC_ADC/Iset: track 20.4 -> 14.1 mm, vias 2 -> 1
- net /Ch1Power/DAC_ADC/Vset: track 20.7 -> 15.1 mm, vias 2 -> 1
- net Net-(U108-VA): track 0.00 -> 5.20 mm
- net Net-(U702-VA): track 0.00 -> 4.44 mm, vias 0 -> 1
- net GND_Ch1: track 48.3 -> 52.1 mm, vias 126 -> 129
- net /Ch1Power1/DAC_ADC/Vset: track 21.6 -> 18.1 mm
- net /Ch1Power1/DAC_ADC/Iset: track 21.2 -> 17.8 mm
- net GND_Ch2: track 48.9 -> 51.9 mm, vias 128 -> 131
- net -1V2Ch2: track 111.5 -> 114.3 mm
- net Net-(U108-VB): track 0.00 -> 2.42 mm
- net Net-(Q501-B): track 9.00 -> 11.0 mm
- net /Ch1Power/Linear_PostReg/OUT+: track 89.4 -> 90.2 mm
- net GNDD: vias 35 -> 34
- net /Ch1Power1/DAC_ADC/SPI_MISO: vias 4 -> 3
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