File: hardware_main/DualPreRegPowerSupply.kicad_pcb (KiCad board)
At the start: 4 copper layers, 99.6 x 100 mm, 375 parts, among them J101 Power Input, J102 Conn_01x03_Pin, J103 Conn_02x02_Odd_Even, J201 Banana_Red, J202 Banana_Black, J203 Conn_02x04_Odd_Even, J204 Conn_02x05_Odd_Even, J205 Conn_01x04_Pin, J402 Banana_Red, J403 Banana_Black, J601 Power Input, J801 Conn_01x03_Pin, J802 Conn_02x02_Odd_Even, J901 Power Input, M401 Fan_4pin, Q101 MMBT3906, Q102 BCP56, Q103 BSS138, Q104 TIP125, Q105 BSS138, Q106 BSS138, Q107 BCP56, Q1401 BSS138, Q301 BCP56, Q302 BSS138, Q303 TIP125, Q304 BCP56, Q501 MMBT3906, Q801 BSS138, Q802 BSS138, Q901 BSS138, U1002 AP7383, U1003 LM2776, U1004 XC6901D121MR-G, U101 TLV4387PWR, U102 ISO6721RFBD, U104 LT8612, U105 LMV331, U106 ATtiny1614-SS, U107 ADS1118IDGS, U108 MCP48FVB22, U109 AP7383, U110 LM2776, U111 XC6901D121MR-G, U1501 LMR51606, U301 TLV4387PWR, U302 LMV331, U501 LT8612, U601 LMR51606, U701 ADS1118IDGS, U702 MCP48FVB22, U801 ISO6721RFBD, U802 ATtiny1614-SS, U901 AP63200WU

Commit message: calc and cleanup
Parts:
- added C1015: 100n, Capacitor_SMD:C_0603_1608Metric, B.Cu at (118.2, 120.2)
- added C1205: 100n, Capacitor_SMD:C_0603_1608Metric, B.Cu at (175.5, 128.8)
- added C1303: 10u, Capacitor_SMD:C_0805_2012Metric, B.Cu at (195.8, 93.4)
- added C808: 10u, Capacitor_SMD:C_0805_2012Metric, B.Cu at (103.2, 98.2)
- C1301, C806: value 4,7u -> 100n
- C1302, C807: value 4,7u -> 27n
- F102, F301: value Fuse -> 3A
- R1301, R807: value 1k -> 12k
- R1302, R808: value 1k -> 10k
Routing:
- net +3V3Ch1: track 32.7 -> 38.9 mm, vias 24 -> 26
- net GND_Ch1: track 52.1 -> 55.9 mm, vias 129 -> 134
- net GND_Ch2: track 51.9 -> 55.3 mm, vias 131 -> 136
- net +3V3Ch2: track 29.6 -> 32.7 mm, vias 24 -> 27
Other:
- board text added: "2 Channel Powersupply V1"
- board text added: "GND 3V3 updi"
- board text added: "updi 3V3 GND"

Commit message: ordering
Parts:
- FL101, FL601: value ACM4520-901-2P-T000 -> DLW5BTM102TQ2L; footprint LibEigen:ACM4520_TDK -> Inductor_SMD:L_CommonModeChoke_Murata_DLW5BTMxxxSQ2x_5x5mm
- moved D104 1.50 mm to (178.5, 53.2)
- moved R134 1.50 mm to (180.1, 53.2)
- moved FL101 0.36 mm to (175.4, 48.9)
- moved FL601 0.10 mm to (114.7, 49.0)
Routing:
- net GND_Ch2: track 55.3 -> 52.9 mm, vias 136 -> 139
- net +40VCh2: track 42.7 -> 43.9 mm
- net GND_Ch1: vias 134 -> 133
