File: hardware_main/Input.kicad_sch (KiCad schematic)
At the start: 11 parts, among them J601 Power Input

Commit message: routing
Parts:
- D602: value LED 40V -> green LED 40V
Changed lines of the file:
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@@
 			)
 		)
-		(property "Value" "LED 40V"
+		(property "Value" "green LED 40V"
 			(at 198.12 112.0774 90)
 			(show_name no)
