File: hardware_main/Input.kicad_sch (KiCad schematic)
At the start: 11 parts, among them J601 Power Input

Commit message: stability calc
Parts:
- C604: value 22u -> 100u
Changed lines of the file:
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@@
 			)
 		)
-		(property "Value" "22u"
+		(property "Value" "100u"
 			(at 182.88 105.7909 0)
 			(show_name no)

Commit message: ordering
Parts:
- FL601: value ACM4520-901-2P-T000 -> DLW5BTM102TQ2L; footprint LibEigen:ACM4520_TDK -> Inductor_SMD:L_CommonModeChoke_Murata_DLW5BTMxxxSQ2x_5x5mm
Changed lines of the file:
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@@
 			)
 		)
-		(property "Value" "ACM4520-901-2P-T000"
+		(property "Value" "DLW5BTM102TQ2L"
 			(at 145.923 110.49 0)
 			(show_name no)
@@
 			)
 		)
-		(property "Footprint" "LibEigen:ACM4520_TDK"
+		(property "Footprint" "Inductor_SMD:L_CommonModeChoke_Murata_DLW5BTMxxxSQ2x_5x5mm"
 			(at 146.05 99.06 0)
 			(hide yes)
