File: hardware_main/MCU.kicad_sch (KiCad schematic)
At the start: 20 parts, among them J801 Conn_01x03_Pin, J802 Conn_02x02_Odd_Even, Q801 BSS138, Q802 BSS138, U801 ISO6721RFBD, U802 ATtiny1614-SS

Commit message: routing
Parts:
- D801, D802: value LED 3V3 -> red LED 3V3
Changed lines of the file:
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@@
 			)
 		)
-		(property "Value" "LED 3V3"
+		(property "Value" "red LED 3V3"
 			(at 163.83 113.3474 90)
 			(show_name no)
@@
 			)
 		)
-		(property "Value" "LED 3V3"
+		(property "Value" "red LED 3V3"
 			(at 234.95 133.6674 90)
 			(show_name no)
