File: hardware_main/Power.kicad_sch (KiCad schematic)
At the start: 28 parts, among them U1002 AP7383, U1003 LM2776, U1004 XC6901D121MR-G, U601 LMR51606

Commit message: routing
Parts:
- D1001: value LED 3V3 -> green LED 3V3
- D1002: value LED -5V -> green LED -5V
Other:
- moved on the sheet: C1001, C1002, C1003, C1005, C1006, C1007, C1008, C1009, C1010, C1011, D1001, D1002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
