File: hardware_main/Power.kicad_sch (KiCad schematic)
At the start: 28 parts, among them U1002 AP7383, U1003 LM2776, U1004 XC6901D121MR-G, U601 LMR51606

Commit message: stability calc
Parts:
- C1001, C1002: value 22u -> 10u
Changed lines of the file:
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@@
 			)
 		)
-		(property "Value" "22u"
+		(property "Value" "10u"
 			(at 77.47 53.34 0)
 			(show_name no)
@@
 			)
 		)
-		(property "Value" "22u"
+		(property "Value" "10u"
 			(at 66.04 53.34 0)
 			(show_name no)

Commit message: calc and cleanup
Changed lines of the file:
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@@
 		(dnp no)
 		(property "Reference" "TP606"
-			(at 199.39 36.83 0)
+			(at 199.39 35.56 0)
 			(show_name no)
 			(do_not_autoplace no)

Commit message: while build
Parts:
- R1004: value ### -> 3,9k
Changed lines of the file:
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@@
 		(fields_autoplaced yes)
 		(property "Reference" "R1004"
-			(at 148.59 118.1101 0)
+			(at 153.67 115.5699 0)
 			(show_name no)
 			(do_not_autoplace no)
@@
 					(size 1.27 1.27)
 				)
-				(justify left)
+				(justify right)
 			)
 		)
-		(property "Value" "###"
-			(at 148.59 115.5701 0)
+		(property "Value" "3,9k"
+			(at 153.67 118.1099 0)
 			(show_name no)
 			(do_not_autoplace no)
@@
 					(size 1.27 1.27)
 				)
-				(justify left)
+				(justify right)
 			)
 		)
