File: hardware_front/Front Panel.kicad_sch (KiCad schematic)
At the start: 47 parts, among them J2 OLED, J3 Conn_02x02_Odd_Even, J4 Conn_02x02_Odd_Even, J5 Conn_02x04_Odd_Even, J6 Conn_01x04, Q401 BSS138, SW1 SW_Push 18mm, SW2 SW_Push 18mm, SW3 SW_Push 18mm, SW4 SW_Push 18mm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

Commit message: routing
Changed lines of the file:
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@@
 	(text "addr\n116 (decimal), 74 (hexadecimal)\n0111 0100"
 		(exclude_from_sim no)
-		(at 186.69 57.15 0)
+		(at 176.53 66.04 0)
 		(effects
 			(font
@@
 	)
 	(junction
+		(at 209.55 80.01)
+		(diameter 0)
+		(color 0 0 0 0)
+	)
+	(junction
 		(at 52.07 157.48)
 		(diameter 0)
@@
 		(color 0 0 0 0)
 	)
-	(junction
-		(at 210.82 80.01)
-		(diameter 0)
-		(color 0 0 0 0)
-	)
 	(no_connect
 		(at 247.65 27.94)
@@
 	(wire
 		(pts
-			(xy 208.28 90.17) (xy 205.74 90.17)
+			(xy 207.01 90.17) (xy 205.74 90.17)
 		)
 		(stroke
@@
 	(wire
 		(pts
-			(xy 210.82 80.01) (xy 212.09 80.01)
-		)
-		(stroke
-			(width 0)
-			(type default)
-		)
-	)
-	(wire
-		(pts
 			(xy 266.7 78.74) (xy 252.73 78.74)
 		)
@@
 	(wire
 		(pts
-			(xy 208.28 80.01) (xy 208.28 90.17)
+			(xy 207.01 80.01) (xy 207.01 90.17)
 		)
 		(stroke
@@
 	(wire
 		(pts
-			(xy 208.28 80.01) (xy 210.82 80.01)
-		)
-		(stroke
-			(width 0)
-			(type default)
-		)
-	)
-	(wire
-		(pts
-			(xy 210.82 78.74) (xy 210.82 80.01)
+			(xy 207.01 80.01) (xy 209.55 80.01)
+		)
+		(stroke
+			(width 0)
+			(type default)
+		)
+	)
+	(wire
+		(pts
+			(xy 209.55 78.74) (xy 209.55 80.01)
+		)
+		(stroke
+			(width 0)
+			(type default)
+		)
+	)
+	(wire
+		(pts
+			(xy 209.55 80.01) (xy 212.09 80.01)
 		)
 		(stroke
@@
 	(symbol
 		(lib_id "power:+3.3V")
-		(at 210.82 78.74 0)
+		(at 209.55 78.74 0)
 		(unit 1)
 		(body_style 1)
@@
 		(fields_autoplaced yes)
 		(property "Reference" "#PWR038"
-			(at 210.82 82.55 0)
+			(at 209.55 82.55 0)
 			(hide yes)
 			(show_name no)
@@
 		)
 		(property "Value" "+3.3V"
-			(at 210.82 73.66 0)
+			(at 209.55 73.66 0)
 			(show_name no)
 			(do_not_autoplace no)
@@
 		)
 		(property "Footprint" ""
-			(at 210.82 78.74 0)
+			(at 209.55 78.74 0)
 			(hide yes)
 			(show_name no)
@@
 		)
 		(property "Datasheet" ""
-			(at 210.82 78.74 0)
+			(at 209.55 78.74 0)
 			(hide yes)
 			(show_name no)
@@
 		)
 		(property "Description" "Power symbol creates a global label with name \"+3.3V\""
-			(at 210.82 78.74 0)
-			(hide yes)
-			(show_name no)
+			(at 209.55 78.74 0)
+			(hide yes)
+			(show_name no)
