File: hardware_front/Front Panel.kicad_sch (KiCad schematic)
At the start: 47 parts, among them J2 OLED, J3 Conn_02x02_Odd_Even, J4 Conn_02x02_Odd_Even, J5 Conn_02x04_Odd_Even, J6 Conn_01x04, Q401 BSS138, SW1 SW_Push 18mm, SW2 SW_Push 18mm, SW3 SW_Push 18mm, SW4 SW_Push 18mm, SW5 SW_Push 18mm, SW7 RotaryEncoder_Switch_MP, SW8 SW_Push 18mm, U3 MCP23008T-E/SS

Commit message: calc and cleanup
Changed lines of the file:
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@@
 		)
 		(property "Value" "MCP23008T-E/SS"
-			(at 190.8967 87.63 0)
+			(at 189.23 85.09 0)
 			(show_name no)
 			(do_not_autoplace no)

Commit message: while build
Parts:
- C5, C7: value C -> 100n
- R15, R16, R17, R18, R19, R20: value xx -> 220
Changed lines of the file:
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@@
 			)
 		)
-		(property "Value" "xx"
+		(property "Value" "220"
 			(at 87.63 163.8299 0)
 			(show_name no)
@@
 			)
 		)
-		(property "Value" "C"
+		(property "Value" "100n"
 			(at 264.16 143.5099 0)
 			(show_name no)
@@
 			)
 		)
-		(property "Value" "xx"
+		(property "Value" "220"
 			(at 24.13 163.8299 0)
 			(show_name no)
@@
 			)
 		)
-		(property "Value" "C"
+		(property "Value" "100n"
 			(at 185.42 129.5399 0)
 			(show_name no)
@@
 			)
 		)
-		(property "Value" "xx"
+		(property "Value" "220"
 			(at 101.6 163.8299 0)
 			(show_name no)
@@
 			)
 		)
-		(property "Value" "xx"
+		(property "Value" "220"
 			(at 54.61 163.8299 0)
 			(show_name no)
@@
 			)
 		)
-		(property "Value" "xx"
+		(property "Value" "220"
 			(at 116.84 163.8299 0)
 			(show_name no)
@@
 			)
 		)
-		(property "Value" "xx"
+		(property "Value" "220"
 			(at 39.37 163.8299 0)
 			(show_name no)
