File: hardware_front/Front Panel.kicad_pcb (KiCad board)
At the start: 4 copper layers, 97.8 x 57.2 mm, 47 parts, among them J2 OLED, J3 Conn_02x02_Odd_Even, J4 Conn_02x02_Odd_Even, J5 Conn_02x04_Odd_Even, J6 Conn_01x04, Q401 BSS138, SW1 SW_Push 18mm, SW2 SW_Push 18mm, SW3 SW_Push 18mm, SW4 SW_Push 18mm, SW5 SW_Push 18mm, SW7 RotaryEncoder_Switch_MP, SW8 SW_Push 18mm, U3 MCP23008T-E/SS

Commit message: calc and cleanup
Changed lines of the file:
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@@
 	)
 	(segment
-		(start 143.5 90)
-		(end 143.5 97.31)
+		(start 143 97.81)
+		(end 138.31 102.5)
 		(width 0.2)
 		(layer "F.Cu")
@@
 	)
 	(segment
-		(start 143.5 97.31)
-		(end 138.31 102.5)
+		(start 143.5 90)
+		(end 143 90.5)
+		(width 0.2)
+		(layer "F.Cu")
+		(net "/ROT_A")
+	)
+	(segment
+		(start 143 90.5)
+		(end 143 97.81)
 		(width 0.2)
 		(layer "F.Cu")
@@
 	)
 	(segment
-		(start 144.3 89.6)
-		(end 144.3 99.4)
-		(width 0.2)
-		(layer "F.Cu")
-		(net "/ROT_B")
-	)
-	(segment
-		(start 145.9 88)
-		(end 144.3 89.6)
+		(start 146.7 88)
+		(end 144.3 90.4)
 		(width 0.2)
 		(layer "F.Cu")
@@
 		(start 144.3 99.4)
 		(end 139.6 104.1)
+		(width 0.2)
+		(layer "F.Cu")
+		(net "/ROT_B")
+	)
+	(segment
+		(start 144.3 90.4)
+		(end 144.3 99.4)
 		(width 0.2)
 		(layer "F.Cu")
@@
 		(width 0.2)
 		(layer "F.Cu")
-		(net "/ROT_B")
-	)
-	(segment
-		(start 146.7 88)
-		(end 145.9 88)
-		(width 0.2)
-		(layer "F.Cu")

Commit message: while build
Parts:
- C5, C7: value C -> 100n
- R15, R16, R17, R18, R19, R20: value xx -> 220
Changed lines of the file:
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@@
 			)
 		)
-		(property "Value" "xx"
+		(property "Value" "220"
 			(at 0 -1.43 90)
 			(layer "B.Fab")
@@
 			)
 		)
-		(property "Value" "xx"
+		(property "Value" "220"
 			(at 0 -1.43 90)
 			(layer "B.Fab")
@@
 			)
 		)
-		(property "Value" "C"
+		(property "Value" "100n"
 			(at 0 -1.43 0)
 			(layer "B.Fab")
@@
 			)
 		)
-		(property "Value" "C"
+		(property "Value" "100n"
 			(at 0 -1.43 90)
 			(layer "B.Fab")
@@
 			)
 		)
-		(property "Value" "xx"
+		(property "Value" "220"
 			(at 0 -1.43 90)
 			(layer "B.Fab")
@@
 			)
 		)
-		(property "Value" "xx"
+		(property "Value" "220"
 			(at 0 -1.43 90)
 			(layer "B.Fab")
@@
 			)
 		)
-		(property "Value" "xx"
+		(property "Value" "220"
 			(at 0 -1.43 90)
 			(layer "B.Fab")
@@
 			)
 		)
-		(property "Value" "xx"
+		(property "Value" "220"
 			(at 0 -1.43 90)
 			(layer "B.Fab")
